Commit message: Manipulator added, only model no extra.

File: mobile_description/urdf/macros.xacro (robot description, xacro)
@@ -1,94 +1,92 @@
 <?xml version="1.0"?>
 <robot xmlns:xacro="http://www.ros.org/wiki/xacro">
-  <xacro:macro name="cylinder_inertia" params="m r h">
-	<inertia
-		ixx="${m*(3*r*r+h*h)/12}"
-		ixy = "0"
-		ixz = "0"
-		iyy="${m*(3*r*r+h*h)/12}"
-		iyz = "0"
-		izz="${m*r*r/2}"
-	/>
-  </xacro:macro>
-  <xacro:macro name="box_inertia" params="m x y z">
-	<inertia
-		ixx="${m*(y*y+z*z)/12}"
-		ixy = "0"
-		ixz = "0"
-		iyy="${m*(x*x+z*z)/12}"
-		iyz = "0"
-		izz="${m*(x*x+z*y)/12}"
-	/>
-  </xacro:macro>
-  <xacro:macro name="sphere_inertia" params="m r">
-	<inertia
-		ixx="${2*m*r*r/5}"
-		ixy = "0"
-		ixz = "0"
-		iyy="${2*m*r*r/5}"
-		iyz = "0"
-		izz="${2*m*r*r/5}"
-	/>
-  </xacro:macro>
-  <xacro:macro name="wheel" params="lr fb Tlr Tfb">
-	<link name="w${lr}${fb}">
-	  <collision>
-		<origin
-			xyz="0 0 0"
+	<xacro:macro name="cylinder_inertia" params="m r h">
+		<inertia
+			ixx="${m*(3*r*r+h*h)/12}"
+			ixy="0"
+			ixz="0"
+			iyy="${m*(3*r*r+h*h)/12}"
+			iyz="0"
+			izz="${m*r*r/2}" />
+	</xacro:macro>
+	<xacro:macro name="box_inertia" params="m x y z">
+		<inertia
+			ixx="${m*(y*y+z*z)/12}"
+			ixy="0"
+			ixz="0"
+			iyy="${m*(x*x+z*z)/12}"
+			iyz="0"
+			izz="${m*(x*x+y*y)/12}" />
+	</xacro:macro>
+	<xacro:macro name="sphere_inertia" params="m r">
+		<inertia
+			ixx="${2*m*r*r/5}"
+			ixy="0"
+			ixz="0"
+			iyy="${2*m*r*r/5}"
+			iyz="0"
+			izz="${2*m*r*r/5}" />
+	</xacro:macro>
+	<xacro:macro name="wheel" params="lr fb Tlr Tfb">
+		<link name="w${lr}${fb}">
+			<inertial>
+				<origin
+					xyz="0 0 0"
+					rpy="0 0 0" />
+				<mass value="${wheelMass}"/>
+				<cylinder_inertia
+					m="${wheelMass}"
+					r="${wheelRadius}"
+					h="${wheelWidth}"/>
+			</inertial>
+			<collision>
+				<origin
+					xyz="0 0 0"
+					rpy="0 0 0" />
+				<geometry>
+					<mesh filename="package://mobile_description/meshes/w${lr}${fb}.STL" />
+				</geometry>
+			</collision>
+			<visual>
+				<origin
+					xyz="0 0 0"
+					rpy="0 0 0" />
+				<geometry>
+					<mesh filename="package://mobile_description/meshes/w${lr}${fb}.STL" />
+				</geometry>
+				<material name="black"/>
+			</visual>
+		</link>
+		<joint name="w${lr}j${fb}" type="continuous">
+			<parent link="chassis"/>
+			<child link="w${lr}${fb}"/>
+			<origin
+				xyz="${Tfb*0.09} ${Tlr*0.1385} ${0.0165+wheelRadius}"
+				rpy="1.5708 0 ${(Tlr+1)*1.5708}" />
+			<axis
+				xyz="0 0 ${Tlr}"
 				rpy="0 0 0" />
-		<geometry>
-		  <mesh filename="package://mobile_description/meshes/w${lr}${fb}.STL" />
-		</geometry>
-	  </collision>
-	  <visual>
-		<origin
-			xyz="0 0 0"
-			rpy="0 0 0" />
-		<geometry>
-		  <mesh filename="package://mobile_description/meshes/w${lr}${fb}.STL" />
-		</geometry>
-			  <material name="black"/>
-	  </visual>
-	  <inertial>
-		<origin
-			xyz="0 0 0"
-				rpy="0 0 0" />
-		<mass value="${wheelMass}"/>
-		<cylinder_inertia
-			m="${wheelMass}"
-			r="${wheelRadius}"
-			h="${wheelWidth}"/>
-	  </inertial>
-	</link>
-	<joint name="w${lr}j${fb}" type="continuous">
-	  <parent link="chassis"/>
-	  <child link="w${lr}${fb}"/>
-	  <origin
-		xyz = "${Tfb*0.09} ${Tlr*0.1385} ${0.0165+wheelRadius}"
-		rpy = "1.5708 0 ${(Tlr+1)*1.5708}" />
-	  <axis xyz="0 0 ${Tlr}"
-	  		  rpy="0 0 0" />
-	  <limit effort="100" velocity="10"/>
-	  <joint_properties damping="0.0" friction="0.0"/>
-	</joint>
-	<gazebo reference="w${lr}${fb}">
-	  <mu1  value="1.0"/>
-	  <mu2  value="1.0"/>
-	  <kp   value="10000000.0"/>
-	  <kd   value="100.0"/>
-	  <minDepth>0.001</minDepth>
-	  <maxVel>1.0</maxVel>
-	  <material>Gazebo/FlatBlack</material>
-	</gazebo>
-	<transmission name="${lr}${fb}_trans">
-	  <type>transmission_interface/SimpleTransmission</type>
-	  <joint name="w${lr}j${fb}">
-		<hardwareInterface>hardware_interface/EffortJointInterface</hardwareInterface>
-	  </joint>
-	  <actuator name="${lr}${fb}Motor">
-		<hardwareInterface>hardware_interface/EffortJointInterface</hardwareInterface>
-		<mechanicalReduction>10</mechanicalReduction>
-	  </actuator>
-	</transmission>
-  </xacro:macro>
+			<limit effort="100" velocity="10"/>
+			<joint_properties damping="0.0" friction="0.0"/>
+		</joint>
+		<gazebo reference="w${lr}${fb}">
+			<mu1 value="1.0"/>
+			<mu2 value="1.0"/>
+			<kp value="10000000.0"/>
+			<kd value="100.0"/>
+			<minDepth>0.001</minDepth>
+			<maxVel>1.0</maxVel>
+			<material>Gazebo/FlatBlack</material>
+		</gazebo>
+		<transmission name="${lr}${fb}_trans">
+			<type>transmission_interface/SimpleTransmission</type>
+			<joint name="w${lr}j${fb}">
+				<hardwareInterface>hardware_interface/EffortJointInterface</hardwareInterface>
+			</joint>
+			<actuator name="${lr}${fb}Motor">
+				<hardwareInterface>hardware_interface/EffortJointInterface</hardwareInterface>
+				<mechanicalReduction>10</mechanicalReduction>
+			</actuator>
+		</transmission>
+	</xacro:macro>
 </robot>

File: mobile_description/urdf/mobile.xacro (robot description, xacro)
@@ -17,19 +17,4 @@
 	<!-- robot chassis -->
 	<link name="chassis">
-		<collision>
-			<origin xyz="0 0 ${wheelRadius}"
-					rpy="0 0 0"/>
-			<geometry>
-				<mesh filename="package://mobile_description/meshes/chassis.STL" />
-			</geometry>
-		</collision>
-		<visual>
-			<origin xyz="0 0 ${wheelRadius}"
-					rpy="0 0 0"/>
-			<geometry>
-				<mesh filename="package://mobile_description/meshes/chassis.STL" />
-			</geometry>
-			<material name="red"/>
-		</visual>
 		<inertial>
 			<origin xyz="0 0 ${wheelRadius}"
@@ -44,4 +29,19 @@
 				izz="0.048521" />
 		</inertial>
+		<visual>
+			<origin xyz="0 0 ${wheelRadius}"
+					rpy="0 0 0"/>
+			<geometry>
+				<mesh filename="package://mobile_description/meshes/chassis.STL" />
+			</geometry>
+			<material name="red"/>
+		</visual>
+		<collision>
+			<origin xyz="0 0 ${wheelRadius}"
+					rpy="0 0 0"/>
+			<geometry>
+				<mesh filename="package://mobile_description/meshes/chassis.STL" />
+			</geometry>
+		</collision>
 	</link>
 	<!-- left-front wheel -->
@@ -53,4 +53,254 @@
 	<!-- right-back wheel -->
 	<wheel lr="r" fb="b" Tlr="-1" Tfb="-1"/>
+	<!-- manipulator base -->
+	<link name="manip_link_base">
+		<inertial>
+			<origin xyz="0 0.0008784 -0.050752" rpy="0 0 0"/>
+			<mass value="0.55594"/>
+			<inertia
+				ixx="0.00781"
+				ixy="0"
+				ixz="0"
+				iyy="0.01091"
+				iyz="-7E-05"
+				izz="0.0032"/>
+		</inertial>
+		<visual>
+			<origin
+				xyz="0 0 0"
+				rpy="0 0 0" />
+			<geometry>
+				<mesh filename="package://mobile_description/meshes/manip_link_base.STL"/>
+			</geometry>
+			<material name="red"/>
+		</visual>
+		<collision>
+			<origin xyz="0 0 0" rpy="0 0 0"/>
+			<geometry>
+				<mesh filename="package://mobile_description/meshes/manip_link_base.STL"/>
+			</geometry>
+		</collision>
+	</link>
+	<joint name="manip_joint_base" type="fixed">
+		<parent link="chassis"/>
+		<child link="manip_link_base"/>
+		<origin xyz="${0.135/2-0.01} 0 ${0.145+0.0165/2-0.005}" rpy="0 0 ${PI/2}"/>
+		<axis xyz="0 0 1"/>
+		<limit effort="0" velocity="0"/>
+	</joint>
+	<link name="manip_link_1">
+		<inertial>
+			<origin
+				xyz="-0.0051711 0.026117 0"
+				rpy="1.5708 0 0" />
+			<mass
+				value="0.19357" />
+			<inertia
+				ixx="0.00064"
+				ixy="-0.0006"
+				ixz="0"
+				iyy="0.00067"
+				iyz="0"
+				izz="0.00104" />
+		</inertial>
+		<visual>
+			<origin
+				xyz="0 0 0"
+				rpy="1.5708 0 0" />
+			<geometry>
+				<mesh filename="package://mobile_description/meshes/manip_link_1.STL"/>
+			</geometry>
+			<material name="orange"/>
+		</visual>
+		<collision>
+			<origin
+				xyz="0 0 0"
+				rpy="1.5708 0 0" />
+			<geometry>
+				<mesh filename="package://mobile_description/meshes/manip_link_1.STL"/>
+			</geometry>
+		</collision>
+	</link>
+	<joint name="manip_joint_1" type="revolute">
+		<parent link="manip_link_base"/>
+		<child link="manip_link_1"/>
+		<origin
+			xyz="0 0 0.018"
+			rpy="0 0 0" />
+		<axis xyz="0 0 1"/>
+		<limit effort="1.0" velocity="1.0" lower="${-3.14}" upper="${3.14}"/>
+	</joint>
+	<link name="manip_link_2">
+		<inertial>
+			<origin
+				xyz="0.0068906 0.13351 -0.00035086"
+				rpy="0 0 0" />
+			<mass
+				value="0.11449" />
+			<inertia
+				ixx="0.0053"
+				ixy="0.00029"
+				ixz="0"
+				iyy="0.00022"
+				iyz="-1E-05"
+				izz="0.00548" />
+		</inertial>
+		<visual>
+			<origin
+				xyz="0 0 0"
+				rpy="0 -1.5708 0" />
+			<geometry>
+				<mesh filename="package://mobile_description/meshes/manip_link_2.STL"/>
+			</geometry>
+			<material name="blue"/>
+		</visual>
+		<collision>
+			<origin
+				xyz="0 0 0"
+				rpy="0 -1.5708 0" />
+			<geometry>
+				<mesh filename="package://mobile_description/meshes/manip_link_2.STL"/>
+			</geometry>
+		</collision>
+	</link>
+	<joint name="manip_joint_2" type="revolute">
+		<parent link="manip_link_1"/>
+		<child link="manip_link_2"/>
+		<origin
+			xyz="0 0 0.05"
+			rpy="1.5708 0 1.5708" />
+		<axis
+			xyz="0 0 1" />
+		<limit effort="1.0" velocity="1.0" lower="${-1.31}" upper="${1.31}"/>
+	</joint>
+	<link name="manip_link_3">
+		<inertial>
+			<origin
+				xyz="0.0054453 0.12903 -0.0002831"
+				rpy="0 0 0" />
+			<mass
+				value="0.11307" />
+			<inertia
+				ixx="0.01892"
+				ixy="0.00037"
+				ixz="0"
+				iyy="0.00016"
+				iyz="-1E-05"
+				izz="0.01905" />
+		</inertial>
+		<visual>
+			<origin
+				xyz="0 0 0"
+				rpy="0 -1.5708 0" />
+			<geometry>
+				<mesh filename="package://mobile_description/meshes/manip_link_3.STL"/>
+			</geometry>
+			<material name="orange"/>
+		</visual>
+		<collision>
+			<origin
+				xyz="0 0 0"
+				rpy="0 0 -1.5708" />
+			<geometry>
+				<mesh filename="package://mobile_description/meshes/manip_link_3.STL"/>
+			</geometry>
+		</collision>
+	</link>
+	<joint name="manip_joint_3" type="revolute">
+		<parent link="manip_link_2"/>
+		<child link="manip_link_3"/>
+		<origin
+			xyz="0 0.205 0"
+			rpy="0 0 0" />
+		<axis
+			xyz="0 0 1" />
+		<limit effort="1.0" velocity="1.0" lower="${-1.31}" upper="${1.31}"/>
+	</joint>
+	<link name="manip_link_4">
+		<inertial>
+			<origin
+				xyz="-0.0094381 0.042624 0"
+				rpy="0 0 0" />
+			<mass
+				value="0.068484" />
+			<inertia
+				ixx="0.01827"
+				ixy="-0.00033"
+				ixz="0"
+				iyy="2E-05"
+				iyz="0"
+				izz="0.01828" />
+		</inertial>
+		<visual>
+			<origin
+				xyz="0 0 0"
+				rpy="0 -1.5708 0" />
+			<geometry>
+				<mesh filename="package://mobile_description/meshes/manip_link_4.STL"/>
+			</geometry>
+			<material name="blue"/>
+		</visual>
+		<collision>
+			<origin
+				xyz="0 0 0"
+				rpy="0 -1.5708 0" />
+			<geometry>
+				<mesh filename="package://mobile_description/meshes/manip_link_4.STL"/>
+			</geometry>
+		</collision>
+	</link>
+	<joint name="manip_joint_4" type="revolute">
+		<parent link="manip_link_3"/>
+		<child link="manip_link_4"/>
+		<origin
+			xyz="0 0.2 0"
+			rpy="0 0 0" />
+		<axis
+			xyz="0 0 1" />
+		<limit effort="1.0" velocity="1.0" lower="${-3.14/2}" upper="${3.14/2}"/>
+	</joint>
+	<link name="manip_link_gripper">
+		<inertial>
+			<origin
+				xyz="0.0019455 0.039335 0.01466"
+				rpy="0 0 0" />
+			<mass
+				value="0.050398" />
+			<inertia
+				ixx="0.0183"
+				ixy="-0.00035"
+				ixz="1E-05"
+				iyy="4E-05"
+				iyz="-0.00044"
+				izz="0.0183" />
+		</inertial>
+		<visual>
+			<origin
+				xyz="0 0 0"
+				rpy="1.5708 0 1.5708" />
+			<geometry>
+				<mesh filename="package://mobile_description/meshes/manip_link_gripper.STL"/>
+			</geometry>
+			<material name="orange"/>
+		</visual>
+		<collision>
+			<origin
+				xyz="0 0 0"
+				rpy="1.5708 0 1.5708" />
+			<geometry>
+				<mesh filename="package://mobile_description/meshes/manip_link_gripper.STL"/>
+			</geometry>
+		</collision>
+	</link>
+	<joint name="manip_joint_gripper" type="revolute">
+		<parent link="manip_link_4"/>
+		<child link="manip_link_gripper"/>
+		<origin
+			xyz="0 0.0895 -0.01"
+			rpy="-1.5708 0 0" />
+		<axis
+			xyz="0 0 1" />
+		<limit effort="1.0" velocity="1.0" lower="${-3.14}" upper="${3.14}"/>
+	</joint>
 	<!-- Sensor models -->
 	<xacro:include filename="$(find mobile_description)/urdf/sensors.xacro" />

File: mobile_description/urdf/mobile_properties.xacro (robot description, xacro)
@@ -18,5 +18,5 @@
 	<xacro:property name="hokuyoWidth" value="0.05"/>
 	<xacro:property name="hokuyoHeight" value="0.07"/>
-	<xacro:property name="hokuyoOffsetX" value="0.14"/>
+	<xacro:property name="hokuyoOffsetX" value="0.17"/>
 	<xacro:property name="hokuyoOffsetZ" value="0.174"/>
 	<!-- Camera properties -->

Commit message: Before reverting to try only mobile for camera issue.

File: mobile_description/urdf/macros.xacro (robot description, xacro)
@@ -32,5 +32,5 @@
 			<inertial>
 				<origin
-					xyz="0 0 0"
+					xyz="0 0 0.005"
 					rpy="0 0 0" />
 				<mass value="${wheelMass}"/>

File: mobile_description/urdf/mobile.xacro (robot description, xacro)
@@ -18,14 +18,14 @@
 	<link name="chassis">
 		<inertial>
-			<origin xyz="0 0 ${wheelRadius}"
+			<origin xyz="0 0 ${wheelRadius+0.035}"
 					rpy="0 0 0"/>
 			<mass value="${chassisMass}"/>
 			<inertia
-				ixx="0.017271"
+				ixx="0.04680"
 				ixy="0"
-				ixz="0"
-				iyy="0.035417"
+				ixz="-0.00022"
+				iyy="0.07212"
 				iyz="0"
-				izz="0.048521" />
+				izz="0.10440" />
 		</inertial>
 		<visual>
@@ -56,13 +56,16 @@
 	<link name="manip_link_base">
 		<inertial>
-			<origin xyz="0 0.0008784 -0.050752" rpy="0 0 0"/>
-			<mass value="0.55594"/>
-			<inertia
-				ixx="0.00781"
-				ixy="0"
-				ixz="0"
-				iyy="0.01091"
-				iyz="-7E-05"
-				izz="0.0032"/>
+			<origin
+				xyz="0 0.05075 0.00088"
+				rpy="0 0 0"/>
+			<mass
+				value="1.50104"/>
+			<inertia
+				ixx="0.01722"
+				ixy="0.0"
+				ixz="0.0"
+				iyy="0.00864"
+				iyz="0.00012"
+				izz="0.02559"/>
 		</inertial>
 		<visual>
@@ -76,5 +79,7 @@
 		</visual>
 		<collision>
-			<origin xyz="0 0 0" rpy="0 0 0"/>
+			<origin
+				xyz="0 0 0"
+				rpy="0 0 0"/>
 			<geometry>
 				<mesh filename="package://mobile_description/meshes/manip_link_base.STL"/>
@@ -92,24 +97,24 @@
 		<inertial>
 			<origin
-				xyz="-0.0051711 0.026117 0"
+				xyz="-0.00517 0.00001 0.02612"
+				rpy="0 0 0" />
+			<mass
+				value="0.19357" />
+			<inertia
+				ixx="0.00071"
+				ixy="-0.00005"
+				ixz="0.0"
+				iyy="0.00181"
+				iyz="0.0"
+				izz="0.00178" />
+		</inertial>
+		<visual>
+			<origin
+				xyz="0 0 0"
 				rpy="1.5708 0 0" />
-			<mass
-				value="0.19357" />
-			<inertia
-				ixx="0.00064"
-				ixy="-0.0006"
-				ixz="0"
-				iyy="0.00067"
-				iyz="0"
-				izz="0.00104" />
-		</inertial>
-		<visual>
-			<origin
-				xyz="0 0 0"
-				rpy="1.5708 0 0" />
 			<geometry>
 				<mesh filename="package://mobile_description/meshes/manip_link_1.STL"/>
 			</geometry>
-			<material name="orange"/>
+			<material name="green"/>
 		</visual>
 		<collision>
@@ -130,19 +135,20 @@
 		<axis xyz="0 0 1"/>
 		<limit effort="1.0" velocity="1.0" lower="${-3.14}" upper="${3.14}"/>
+    	<dynamics damping="0.7"/>
 	</joint>
 	<link name="manip_link_2">
 		<inertial>
 			<origin
-				xyz="0.0068906 0.13351 -0.00035086"
-				rpy="0 0 0" />
-			<mass
-				value="0.11449" />
-			<inertia
-				ixx="0.0053"
-				ixy="0.00029"
-				ixz="0"
-				iyy="0.00022"
-				iyz="-1E-05"
-				izz="0.00548" />
+				xyz="0.00000 0.13351 -0.00035"
+				rpy="0 -1.5708 0" />
+			<mass
+				value="0.30912" />
+			<inertia
+				ixx="0.00177"
+				ixy="0.00036"
+				ixz="0.0"
+				iyy="0.00057"
+				iyz="0.0"
+				izz="0.00224" />
 		</inertial>
 		<visual>
@@ -172,20 +178,21 @@
 		<axis
 			xyz="0 0 1" />
-		<limit effort="1.0" velocity="1.0" lower="${-1.31}" upper="${1.31}"/>
+		<limit effort="1.0" velocity="1.0" lower="${-PI/2}" upper="${PI/2}"/>
+    	<dynamics damping="0.7"/>
 	</joint>
 	<link name="manip_link_3">
 		<inertial>
 			<origin
-				xyz="0.0054453 0.12903 -0.0002831"
-				rpy="0 0 0" />
-			<mass
-				value="0.11307" />
-			<inertia
-				ixx="0.01892"
-				ixy="0.00037"
-				ixz="0"
-				iyy="0.00016"
-				iyz="-1E-05"
-				izz="0.01905" />
+				xyz="0.00000 0.12903 -0.00028"
+				rpy="0 -1.5708 0" />
+			<mass
+				value="0.30530" />
+			<inertia
+				ixx="0.00175"
+				ixy="0.00032"
+				ixz="0.0"
+				iyy="0.00042"
+				iyz="0.0"
+				izz="0.00208" />
 		</inertial>
 		<visual>
@@ -196,10 +203,10 @@
 				<mesh filename="package://mobile_description/meshes/manip_link_3.STL"/>
 			</geometry>
-			<material name="orange"/>
-		</visual>
-		<collision>
-			<origin
-				xyz="0 0 0"
-				rpy="0 0 -1.5708" />
+			<material name="green"/>
+		</visual>
+		<collision>
+			<origin
+				xyz="0 0 0"
+				rpy="0 -1.5708 0" />
 			<geometry>
 				<mesh filename="package://mobile_description/meshes/manip_link_3.STL"/>
@@ -215,20 +222,21 @@
 		<axis
 			xyz="0 0 1" />
-		<limit effort="1.0" velocity="1.0" lower="${-1.31}" upper="${1.31}"/>
+		<limit effort="1.0" velocity="1.0" lower="${-PI}" upper="${PI}"/>
+    	<dynamics damping="0.7"/>
 	</joint>
 	<link name="manip_link_4">
 		<inertial>
 			<origin
-				xyz="-0.0094381 0.042624 0"
-				rpy="0 0 0" />
-			<mass
-				value="0.068484" />
-			<inertia
-				ixx="0.01827"
-				ixy="-0.00033"
-				ixz="0"
-				iyy="2E-05"
-				iyz="0"
-				izz="0.01828" />
+				xyz="0.00000 0.04262 -0.00944"
+				rpy="0 -1.5708 0" />
+			<mass
+				value="0.18491" />
+			<inertia
+				ixx="0.00017"
+				ixy="0.0"
+				ixz="0.0"
+				iyy="0.00005"
+				iyz="0.0"
+				izz="0.00018" />
 		</inertial>
 		<visual>
@@ -258,29 +266,30 @@
 		<axis
 			xyz="0 0 1" />
-		<limit effort="1.0" velocity="1.0" lower="${-3.14/2}" upper="${3.14/2}"/>
+		<limit effort="1.0" velocity="1.0" lower="${-PI}" upper="${PI}"/>
+    	<dynamics damping="0.7"/>
 	</joint>
 	<link name="manip_link_gripper">
 		<inertial>
 			<origin
-				xyz="0.0019455 0.039335 0.01466"
-				rpy="0 0 0" />
-			<mass
-				value="0.050398" />
-			<inertia
-				ixx="0.0183"
-				ixy="-0.00035"
-				ixz="1E-05"
-				iyy="4E-05"
-				iyz="-0.00044"
-				izz="0.0183" />
-		</inertial>
-		<visual>
-			<origin
-				xyz="0 0 0"
+				xyz="0.01466 0.00195 0.03933"
 				rpy="1.5708 0 1.5708" />
+			<mass
+				value="0.13607" />
+			<inertia
+				ixx="0.00010"
+				ixy="0.0"
+				ixz="0.0"
+				iyy="0.00006"
+				iyz="-0.00002"
+				izz="0.00010" />
+		</inertial>
+		<visual>
+			<origin
+				xyz="0 0 0"
+				rpy="1.5708 0 1.5708" />
 			<geometry>
 				<mesh filename="package://mobile_description/meshes/manip_link_gripper.STL"/>
 			</geometry>
-			<material name="orange"/>
+			<material name="green"/>
 		</visual>
 		<collision>
@@ -293,5 +302,5 @@
 		</collision>
 	</link>
-	<joint name="manip_joint_gripper" type="revolute">
+	<joint name="manip_joint_5" type="revolute">
 		<parent link="manip_link_4"/>
 		<child link="manip_link_gripper"/>
@@ -302,4 +311,5 @@
 			xyz="0 0 1" />
 		<limit effort="1.0" velocity="1.0" lower="${-3.14}" upper="${3.14}"/>
+    	<dynamics damping="0.7"/>
 	</joint>
 	<!-- Sensor models -->

File: mobile_description/urdf/mobile_properties.xacro (robot description, xacro)
@@ -7,5 +7,5 @@
 	<xacro:property name="chassisLength" value="0.40"/>
 	<xacro:property name="chassisWidth" value="0.27"/>
-	<xacro:property name="chassisMass" value="2.5"/>
+	<xacro:property name="chassisMass" value="5.0"/>
 	<!-- Differential-drive wheels properties -->
 	<xacro:property name="wheelWidth" value="0.026"/>
@@ -25,5 +25,5 @@
 	<xacro:property name="cameraHeight" value="0.03"/>
 	<xacro:property name="cameraMass" value="0.01"/>
-	<xacro:property name="cameraOffsetX" value="0.178"/>
-	<xacro:property name="cameraOffsetZ" value="0.122"/>
+	<xacro:property name="cameraOffsetX" value="0.18"/>
+	<xacro:property name="cameraOffsetZ" value="0.1222"/>
 </robot>

Commit message: Adde my_controller_pkg, and created a working custom controller.

File: mobile_description/urdf/macros.xacro (robot description, xacro)
@@ -86,5 +86,5 @@
 			<actuator name="${lr}${fb}Motor">
 				<hardwareInterface>hardware_interface/EffortJointInterface</hardwareInterface>
-				<mechanicalReduction>10</mechanicalReduction>
+				<mechanicalReduction>2</mechanicalReduction>
 			</actuator>
 		</transmission>

File: mobile_description/urdf/mobile.xacro (robot description, xacro)
@@ -20,20 +20,12 @@
 			<origin xyz="0 0 ${wheelRadius+0.035}"
 					rpy="0 0 0"/>
-			<mass value="15.0"/>
+			<mass value="12.0"/>
 			<inertia
-				ixx="0.017271"
+				ixx="0.04680"
 				ixy="0"
-				ixz="0"
-				iyy="0.035417"
+				ixz="-0.00022"
+				iyy="0.07212"
 				iyz="0"
-				izz="0.048521" />
-			<!-- <inertia
-				ixx="1.0"
-				ixy="0.00000"
-				ixz="0.00000"
-				iyy="1.0"
-				iyz="0.00000"
-				izz="1.0" /> -->
-			<!-- <box_inertia m="40" x="0.40" y="0.27" z="0.10" /> -->
+				izz="0.10440" />
 		</inertial>
 		<visual>
@@ -62,5 +54,5 @@
 	<wheel lr="r" fb="b" Tlr="-1" Tfb="-1"/>
 	<!-- Arm models -->
-	<!-- <xacro:include filename="$(find mobile_description)/urdf/arm.xacro" /> -->
+	<xacro:include filename="$(find mobile_description)/urdf/arm.xacro" />
 	<!-- Sensor models -->
 	<xacro:include filename="$(find mobile_description)/urdf/sensors.xacro" />

Commit message: Updated controller header files for document generation.
Fixes:
- Velocity limits increased for mobile base wheel joints.

To Do:
- Create an action file to follow a trejactory for mobile base.
- Create an action file to command arm positions.

Signed-off-by: Fatih Kaan AKKUS <fthknakkus@hotmail.com>

File: mobile_description/urdf/macros.xacro (robot description, xacro)
@@ -67,5 +67,5 @@
 				xyz="0 0 ${Tlr}"
 				rpy="0 0 0" />
-			<limit effort="6.0" velocity="5.0"/>
+			<limit effort="100.0" velocity="100.0"/>
 			<joint_properties damping="0.0" friction="0.0"/>
 		</joint>
