Commit message: my_filter_pkg introduced. Controller updates.
Signed-off-by: Fatih Kaan AKKUS <fthknakkus@hotmail.com>

File: mobile_description/urdf/arm.xacro (robot description, xacro)
@@ -92,5 +92,5 @@
 	<joint
 		name="m_joint_1"
-		type="revolute">
+		type="continuous">
 		<origin
 			xyz="0 0 0.018"
@@ -102,9 +102,9 @@
 		<axis
 			xyz="0 0 1" />
-		<limit
-			effort="10.0"
-			velocity="1.0"
-			lower="${-3.14}"
-			upper="${3.14}"/>
+		<!-- <limit
+			effort="10.0"
+			velocity="1.0"/> -->
+			<!-- lower="${-3.14}"
+			upper="${3.14}" -->
 	</joint>
 	<link

Commit message: Created MobileController. Updated other controllers.
- Lots of fixes.
- Lots of updated.

Signed-off-by: Fatih Kaan AKKUS <fthknakkus@hotmail.com>

File: mobile_description/urdf/arm.xacro (robot description, xacro)
@@ -92,5 +92,5 @@
 	<joint
 		name="m_joint_1"
-		type="continuous">
+		type="revolute">
 		<origin
 			xyz="0 0 0.018"
@@ -102,9 +102,9 @@
 		<axis
 			xyz="0 0 1" />
-		<!-- <limit
-			effort="10.0"
-			velocity="1.0"/> -->
-			<!-- lower="${-3.14}"
-			upper="${3.14}" -->
+		<limit
+			effort="6.0"
+			velocity="1.0"
+			lower="${-3.14}"
+			upper="${3.14}" />
 	</joint>
 	<link
@@ -161,5 +161,5 @@
 			xyz="0 0 1" />
 		<limit
-			effort="10.0"
+			effort="6.0"
 			velocity="1.0"
 			lower="${-3.14}"
@@ -219,5 +219,5 @@
 			xyz="0 0 1" />
 		<limit
-			effort="10.0"
+			effort="6.0"
 			velocity="1.0"
 			lower="${-3.14}"
@@ -277,5 +277,5 @@
 			xyz="0 0 1" />
 		<limit
-			effort="10.0"
+			effort="6.0"
 			velocity="1.0"
 			lower="${-3.14}"
@@ -335,5 +335,5 @@
 			xyz="0 0 1" />
 		<limit
-			effort="10.0"
+			effort="6.0"
 			velocity="1.0"
 			lower="${-3.14}"

File: mobile_description/urdf/macros.xacro (robot description, xacro)
@@ -67,14 +67,14 @@
 				xyz="0 0 ${Tlr}"
 				rpy="0 0 0" />
-			<limit effort="100" velocity="10"/>
+			<limit effort="6.0" velocity="5.0"/>
 			<joint_properties damping="0.0" friction="0.0"/>
 		</joint>
 		<gazebo reference="w${lr}${fb}">
-			<mu1 value="1.0"/>
-			<mu2 value="1.0"/>
-			<kp value="10000000.0"/>
-			<kd value="100.0"/>
+			<mu1 value="100.0"/>
+			<mu2 value="100.0"/>
+			<kp value="1.0E+6"/>
+			<kd value="1.0E+0"/>
 			<minDepth>0.001</minDepth>
-			<maxVel>1.0</maxVel>
+			<maxVel>100.0</maxVel>
 			<material>Gazebo/FlatBlack</material>
 		</gazebo>
@@ -82,9 +82,9 @@
 			<type>transmission_interface/SimpleTransmission</type>
 			<joint name="w${lr}j${fb}">
-				<hardwareInterface>hardware_interface/EffortJointInterface</hardwareInterface>
+				<hardwareInterface>hardware_interface/VelocityJointInterface</hardwareInterface>
 			</joint>
 			<actuator name="${lr}${fb}Motor">
-				<hardwareInterface>hardware_interface/EffortJointInterface</hardwareInterface>
-				<mechanicalReduction>2</mechanicalReduction>
+				<hardwareInterface>hardware_interface/VelocityJointInterface</hardwareInterface>
+				<mechanicalReduction>10</mechanicalReduction>
 			</actuator>
 		</transmission>
