Commit message: Added simple gripper, replaced \t's with spaces in all docs.
Signed-off-by: Fatih Kaan AKKUS <fthknakkus@hotmail.com>

File: mobile_description/urdf/arm.xacro (robot description, xacro)
@@ -1,351 +1,491 @@
 <?xml version="1.0" ?>
 <robot xmlns:xacro="http://www.ros.org/wiki/xacro">
-	<link
-		name="m_base">
-		<inertial>
-			<origin
-				xyz="-3.4809E-08 -0.05038 0.0010533"
-				rpy="0 0 0" />
-			<mass
-				value="1.5121" />
-			<inertia
-				ixx="0.0006372"
-				ixy="2.6122E-09"
-				ixz="1.9384E-10"
-				iyy="0.00027925"
-				iyz="0.00011021"
-				izz="0.00064253" />
-		</inertial>
-		<visual>
-			<origin
-				xyz="0 0 0"
-				rpy="0 0 0" />
-			<geometry>
-				<mesh
-					filename="package://mobile_description/meshes/m_base.STL" />
-			</geometry>
-			<material
-				name="">
-				<color
-					rgba="0.75294 0.75294 0.75294 1" />
-			</material>
-		</visual>
-		<collision>
-			<origin
-				xyz="0 0 0"
-				rpy="0 0 0" />
-			<geometry>
-				<mesh
-					filename="package://mobile_description/meshes/m_base.STL" />
-			</geometry>
-		</collision>
-	</link>
-	<joint name="m_joint_base" type="fixed">
-		<parent link="chassis"/>
-		<child link="m_base"/>
-		<origin
-			xyz="${0.135/2-0.01} 0 ${0.145+0.0165/2-0.005}"
-			rpy="0 0 ${-PI/2}"/>
-		<axis xyz="0 0 0"/>
-		<limit effort="0" velocity="0"/>
-	</joint>
-	<link
-		name="m_link_1">
-		<inertial>
-			<origin
-				xyz="5.3086E-06 -0.0050977 0.025693"
-				rpy="0 0 0" />
-			<mass
-				value="0.53016" />
-			<inertia
-				ixx="0.0013772"
-				ixy="1.2464E-07"
-				ixz="6.5275E-08"
-				iyy="0.000284"
-				iyz="5.4578E-05"
-				izz="0.0010934" />
-		</inertial>
-		<visual>
-			<origin
-				xyz="0 0 0"
-				rpy="0 0 0" />
-			<geometry>
-				<mesh
-					filename="package://mobile_description/meshes/m_link_1.STL" />
-			</geometry>
-			<material
-				name="">
-				<color
-					rgba="0.75294 0.75294 0.75294 1" />
-			</material>
-		</visual>
-		<collision>
-			<origin
-				xyz="0 0 0"
-				rpy="0 0 0" />
-			<geometry>
-				<mesh
-					filename="package://mobile_description/meshes/m_link_1.STL" />
-			</geometry>
-		</collision>
-	</link>
-	<joint
-		name="m_joint_1"
-		type="revolute">
-		<origin
-			xyz="0 0 0.018"
-			rpy="9.5272E-17 2.5487E-17 -1.5708" />
-		<parent
-			link="m_base" />
-		<child
-			link="m_link_1" />
-		<axis
-			xyz="0 0 1" />
-		<limit
-			effort="6.0"
-			velocity="1.0"
-			lower="${-3.14}"
-			upper="${3.14}" />
-	</joint>
-	<link
-		name="m_link_2">
-		<inertial>
-			<origin
-				xyz="0.12595 0.00091717 -0.005421"
-				rpy="0 0 0" />
-			<mass
-				value="0.33957" />
-			<inertia
-				ixx="0.00053588"
-				ixy="8.0811E-06"
-				ixz="0.00037406"
-				iyy="0.0014491"
-				iyz="-4.6471E-06"
-				izz="0.00095056" />
-		</inertial>
-		<visual>
-			<origin
-				xyz="0 0 0"
-				rpy="0 0 0" />
-			<geometry>
-				<mesh
-					filename="package://mobile_description/meshes/m_link_2.STL" />
-			</geometry>
-			<material
-				name="">
-				<color
-					rgba="0.75294 0.75294 0.75294 1" />
-			</material>
-		</visual>
-		<collision>
-			<origin
-				xyz="0 0 0"
-				rpy="0 0 0" />
-			<geometry>
-				<mesh
-					filename="package://mobile_description/meshes/m_link_2.STL" />
-			</geometry>
-		</collision>
-	</link>
-	<joint
-		name="m_joint_2"
-		type="revolute">
-		<origin
-			xyz="0 0 0.055"
-			rpy="1.5708 -1.5708 0" />
-		<parent
-			link="m_link_1" />
-		<child
-			link="m_link_2" />
-		<axis
-			xyz="0 0 1" />
-		<limit
-			effort="6.0"
-			velocity="1.0"
-			lower="${-3.14}"
-			upper="${3.14}"/>
-	</joint>
-	<link
-		name="m_link_3">
-		<inertial>
-			<origin
-				xyz="0.12805 0.00074276 -0.0046757"
-				rpy="0 0 0" />
-			<mass
-				value="0.32588" />
-			<inertia
-				ixx="0.00038507"
-				ixy="6.7854E-06"
-				ixz="0.00031809"
-				iyy="0.0012115"
-				iyz="-3.4316E-06"
-				izz="0.0008557" />
-		</inertial>
-		<visual>
-			<origin
-				xyz="0 0 0"
-				rpy="0 0 0" />
-			<geometry>
-				<mesh
-					filename="package://mobile_description/meshes/m_link_3.STL" />
-			</geometry>
-			<material
-				name="">
-				<color
-					rgba="0.75294 0.75294 0.75294 1" />
-			</material>
-		</visual>
-		<collision>
-			<origin
-				xyz="0 0 0"
-				rpy="0 0 0" />
-			<geometry>
-				<mesh
-					filename="package://mobile_description/meshes/m_link_3.STL" />
-			</geometry>
-		</collision>
-	</link>
-	<joint
-		name="m_joint_3"
-		type="revolute">
-		<origin
-			xyz="0.2 0 0"
-			rpy="4.4409E-16 4.5852E-16 -1.7798E-16" />
-		<parent
-			link="m_link_2" />
-		<child
-			link="m_link_3" />
-		<axis
-			xyz="0 0 1" />
-		<limit
-			effort="6.0"
-			velocity="1.0"
-			lower="${-3.14}"
-			upper="${3.14}"/>
-	</joint>
-	<link
-		name="m_link_4">
-		<inertial>
-			<origin
-				xyz="0.042624 1.8551E-17 0.0094381"
-				rpy="0 0 0" />
-			<mass
-				value="0.18491" />
-			<inertia
-				ixx="9.4388E-07"
-				ixy="-1.361E-20"
-				ixz="-2.8787E-07"
-				iyy="4.3712E-05"
-				iyz="-9.3643E-23"
-				izz="4.2768E-05" />
-		</inertial>
-		<visual>
-			<origin
-				xyz="0 0 0"
-				rpy="0 0 0" />
-			<geometry>
-				<mesh
-					filename="package://mobile_description/meshes/m_link_4.STL" />
-			</geometry>
-			<material
-				name="">
-				<color
-					rgba="0.75294 0.75294 0.75294 1" />
-			</material>
-		</visual>
-		<collision>
-			<origin
-				xyz="0 0 0"
-				rpy="0 0 0" />
-			<geometry>
-				<mesh
-					filename="package://mobile_description/meshes/m_link_4.STL" />
-			</geometry>
-		</collision>
-	</link>
-	<joint
-		name="m_joint_4"
-		type="revolute">
-		<origin
-			xyz="0.2 0 0"
-			rpy="-3.3307E-16 -6.6356E-16 -1.9531E-16" />
-		<parent
-			link="m_link_3" />
-		<child
-			link="m_link_4" />
-		<axis
-			xyz="0 0 1" />
-		<limit
-			effort="6.0"
-			velocity="1.0"
-			lower="${-3.14}"
-			upper="${3.14}"/>
-	</joint>
-	<link
-		name="m_link_gripper">
-		<inertial>
-			<origin
-				xyz="-0.0069546 0.0010309 -0.036727"
-				rpy="0 0 0" />
-			<mass
-				value="0.098787" />
-			<inertia
-				ixx="5.8957E-05"
-				ixy="1.4882E-06"
-				ixz="5.6679E-06"
-				iyy="6.3174E-05"
-				iyz="-4.7843E-07"
-				izz="2.5215E-05" />
-		</inertial>
-		<visual>
-			<origin
-				xyz="0 0 0"
-				rpy="0 0 0" />
-			<geometry>
-				<mesh
-					filename="package://mobile_description/meshes/m_link_gripper.STL" />
-			</geometry>
-			<material
-				name="">
-				<color
-					rgba="0.75294 0.75294 0.75294 1" />
-			</material>
-		</visual>
-		<collision>
-			<origin
-				xyz="0 0 0"
-				rpy="0 0 0" />
-			<geometry>
-				<mesh
-					filename="package://mobile_description/meshes/m_link_gripper.STL" />
-			</geometry>
-		</collision>
-	</link>
-	<joint
-		name="m_joint_5"
-		type="revolute">
-		<origin
-			xyz="0.0895 0 0.0095"
-			rpy="1.5708 3.861E-32 -1.5708" />
-		<parent
-			link="m_link_4" />
-		<child
-			link="m_link_gripper" />
-		<axis
-			xyz="0 0 1" />
-		<limit
-			effort="6.0"
-			velocity="1.0"
-			lower="${-3.14}"
-			upper="${3.14}"/>
-	</joint>
-	<!-- Arm @ Gazebo -->
-	<xacro:include filename="$(find mobile_description)/urdf/arm.gazebo" />
+    <link
+        name="m_base">
+        <inertial>
+            <origin
+                xyz="-3.4809E-08 -0.05038 0.0010533"
+                rpy="0 0 0" />
+            <mass
+                value="1.5121" />
+            <inertia
+                ixx="0.0006372"
+                ixy="2.6122E-09"
+                ixz="1.9384E-10"
+                iyy="0.00027925"
+                iyz="0.00011021"
+                izz="0.00064253" />
+        </inertial>
+        <visual>
+            <origin
+                xyz="0 0 0"
+                rpy="0 0 0" />
+            <geometry>
+                <mesh
+                    filename="package://mobile_description/meshes/m_base.STL" />
+            </geometry>
+            <material
+                name="">
+                <color
+                    rgba="0.75294 0.75294 0.75294 1" />
+            </material>
+        </visual>
+        <collision>
+            <origin
+                xyz="0 0 0"
+                rpy="0 0 0" />
+            <geometry>
+                <mesh
+                    filename="package://mobile_description/meshes/m_base.STL" />
+            </geometry>
+        </collision>
+    </link>
+    <joint name="m_joint_base" type="fixed">
+        <parent link="chassis"/>
+        <child link="m_base"/>
+        <origin
+            xyz="${0.135/2-0.01} 0 ${0.145+0.0165/2-0.005}"
+            rpy="0 0 ${-PI/2}"/>
+        <axis xyz="0 0 0"/>
+        <limit effort="0" velocity="0"/>
+    </joint>
+    <link
+        name="m_link_1">
+        <inertial>
+            <origin
+                xyz="5.3086E-06 -0.0050977 0.025693"
+                rpy="0 0 0" />
+            <mass
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
File: mobile_description/urdf/macros.xacro (robot description, xacro)
@@ -1,92 +1,92 @@
 <?xml version="1.0"?>
 <robot xmlns:xacro="http://www.ros.org/wiki/xacro">
-	<xacro:macro name="cylinder_inertia" params="m r h">
-		<inertia
-			ixx="${m*(3*r*r+h*h)/12}"
-			ixy="0"
-			ixz="0"
-			iyy="${m*(3*r*r+h*h)/12}"
-			iyz="0"
-			izz="${m*r*r/2}" />
-	</xacro:macro>
-	<xacro:macro name="box_inertia" params="m x y z">
-		<inertia
-			ixx="${m*(y*y+z*z)/12}"
-			ixy="0"
-			ixz="0"
-			iyy="${m*(x*x+z*z)/12}"
-			iyz="0"
-			izz="${m*(x*x+y*y)/12}" />
-	</xacro:macro>
-	<xacro:macro name="sphere_inertia" params="m r">
-		<inertia
-			ixx="${2*m*r*r/5}"
-			ixy="0"
-			ixz="0"
-			iyy="${2*m*r*r/5}"
-			iyz="0"
-			izz="${2*m*r*r/5}" />
-	</xacro:macro>
-	<xacro:macro name="wheel" params="lr fb Tlr Tfb">
-		<link name="w${lr}${fb}">
-			<inertial>
-				<origin
-					xyz="0 0 0.005"
-					rpy="0 0 0" />
-				<mass value="${wheelMass}"/>
-				<cylinder_inertia
-					m="${wheelMass}"
-					r="${wheelRadius}"
-					h="${wheelWidth}"/>
-			</inertial>
-			<collision>
-				<origin
-					xyz="0 0 0"
-					rpy="0 0 0" />
-				<geometry>
-					<mesh filename="package://mobile_description/meshes/w${lr}${fb}.STL" />
-				</geometry>
-			</collision>
-			<visual>
-				<origin
-					xyz="0 0 0"
-					rpy="0 0 0" />
-				<geometry>
-					<mesh filename="package://mobile_description/meshes/w${lr}${fb}.STL" />
-				</geometry>
-				<material name="black"/>
-			</visual>
-		</link>
-		<joint name="w${lr}j${fb}" type="continuous">
-			<parent link="chassis"/>
-			<child link="w${lr}${fb}"/>
-			<origin
-				xyz="${Tfb*0.09} ${Tlr*0.1385} ${0.0165+wheelRadius}"
-				rpy="1.5708 0 ${(Tlr+1)*1.5708}" />
-			<axis
-				xyz="0 0 ${Tlr}"
-				rpy="0 0 0" />
-			<limit effort="100.0" velocity="100.0"/>
-			<joint_properties damping="0.0" friction="0.0"/>
-		</joint>
-		<gazebo reference="w${lr}${fb}">
-			<mu1 value="1.2"/>
-			<mu2 value="1.2"/>
-			<kp value="1.0E+6"/>
-			<kd value="1.0E+0"/>
-			<minDepth>0.001</minDepth>
-			<maxVel>100.0</maxVel>
-			<material>Gazebo/FlatBlack</material>
-		</gazebo>
-		<transmission name="${lr}${fb}_trans">
-			<type>transmission_interface/SimpleTransmission</type>
-			<joint name="w${lr}j${fb}">
-				<hardwareInterface>hardware_interface/VelocityJointInterface</hardwareInterface>
-			</joint>
-			<actuator name="${lr}${fb}Motor">
-				<hardwareInterface>hardware_interface/VelocityJointInterface</hardwareInterface>
-				<mechanicalReduction>10</mechanicalReduction>
-			</actuator>
-		</transmission>
-	</xacro:macro>
+    <xacro:macro name="cylinder_inertia" params="m r h">
+        <inertia
+            ixx="${m*(3*r*r+h*h)/12}"
+            ixy="0"
+            ixz="0"
+            iyy="${m*(3*r*r+h*h)/12}"
+            iyz="0"
+            izz="${m*r*r/2}" />
+    </xacro:macro>
+    <xacro:macro name="box_inertia" params="m x y z">
+        <inertia
+            ixx="${m*(y*y+z*z)/12}"
+            ixy="0"
+            ixz="0"
+            iyy="${m*(x*x+z*z)/12}"
+            iyz="0"
+            izz="${m*(x*x+y*y)/12}" />
+    </xacro:macro>
+    <xacro:macro name="sphere_inertia" params="m r">
+        <inertia
+            ixx="${2*m*r*r/5}"
+            ixy="0"
+            ixz="0"
+            iyy="${2*m*r*r/5}"
+            iyz="0"
+            izz="${2*m*r*r/5}" />
+    </xacro:macro>
+    <xacro:macro name="wheel" params="lr fb Tlr Tfb">
+        <link name="w${lr}${fb}">
+            <inertial>
+                <origin
+                    xyz="0 0 0.005"
+                    rpy="0 0 0" />
+                <mass value="${wheelMass}"/>
+                <cylinder_inertia
+                    m="${wheelMass}"
+                    r="${wheelRadius}"
+                    h="${wheelWidth}"/>
+            </inertial>
+            <collision>
+                <origin
+                    xyz="0 0 0"
+                    rpy="0 0 0" />
+                <geometry>
+                    <mesh filename="package://mobile_description/meshes/w${lr}${fb}.STL" />
+                </geometry>
+            </collision>
+            <visual>
+                <origin
+                    xyz="0 0 0"
+                    rpy="0 0 0" />
+                <geometry>
+                    <mesh filename="package://mobile_description/meshes/w${lr}${fb}.STL" />
+                </geometry>
+                <material name="black"/>
+            </visual>
+        </link>
+        <joint name="w${lr}j${fb}" type="continuous">
+            <parent link="chassis"/>
+            <child link="w${lr}${fb}"/>
+            <origin
+                xyz="${Tfb*0.09} ${Tlr*0.1385} ${0.0165+wheelRadius}"
+                rpy="1.5708 0 ${(Tlr+1)*1.5708}" />
+            <axis
+                xyz="0 0 ${Tlr}"
+                rpy="0 0 0" />
+            <limit effort="100.0" velocity="100.0"/>
+            <joint_properties damping="0.0" friction="0.0"/>
+        </joint>
+        <gazebo reference="w${lr}${fb}">
+            <mu1 value="1.2"/>
+            <mu2 value="1.2"/>
+            <kp value="1.0E+6"/>
+            <kd value="1.0E+0"/>
+            <minDepth>0.001</minDepth>
+            <maxVel>100.0</maxVel>
+            <material>Gazebo/FlatBlack</material>
+        </gazebo>
+        <transmission name="${lr}${fb}_trans">
+            <type>transmission_interface/SimpleTransmission</type>
+            <joint name="w${lr}j${fb}">
+                <hardwareInterface>hardware_interface/VelocityJointInterface</hardwareInterface>
+            </joint>
+            <actuator name="${lr}${fb}Motor">
+                <hardwareInterface>hardware_interface/VelocityJointInterface</hardwareInterface>
+                <mechanicalReduction>10</mechanicalReduction>
+            </actuator>
+        </transmission>
+    </xacro:macro>
 </robot>

File: mobile_description/urdf/materials.xacro (robot description, xacro)
@@ -1,33 +1,33 @@
 <?xml version="1.0"?>
 <robot>
-	<material name="black">
-		<color rgba="0.0 0.0 0.0 1.0"/>
-	</material>
-	<material name="blue">
-		<color rgba="0.0 0.0 0.8 1.0"/>
-	</material>
-	<material name="green">
-		<color rgba="0.0 0.8 0.0 1.0"/>
-	</material>
-	<material name="grey">
-		<color rgba="0.2 0.2 0.2 1.0"/>
-	</material>
-	<material name="light_grey">
-		<color rgba="0.6 0.6 0.6 1"/>
-	</material>
-	<material name="dark_grey">
-		<color rgba="0.3 0.3 0.3 1"/>
-	</material>
-	<material name="orange">
-		<color rgba="${255/255} ${108/255} ${10/255} 1.0"/>
-	</material>
-	<material name="brown">
-		<color rgba="${222/255} ${207/255} ${195/255} 1.0"/>
-	</material>
-	<material name="red">
-		<color rgba="0.8 0.0 0.0 1.0"/>
-	</material>
-	<material name="white">
-		<color rgba="1.0 1.0 1.0 1.0"/>
-	</material>
+    <material name="black">
+        <color rgba="0.0 0.0 0.0 1.0"/>
+    </material>
+    <material name="blue">
+        <color rgba="0.0 0.0 0.8 1.0"/>
+    </material>
+    <material name="green">
+        <color rgba="0.0 0.8 0.0 1.0"/>
+    </material>
+    <material name="grey">
+        <color rgba="0.2 0.2 0.2 1.0"/>
+    </material>
+    <material name="light_grey">
+        <color rgba="0.6 0.6 0.6 1"/>
+    </material>
+    <material name="dark_grey">
+        <color rgba="0.3 0.3 0.3 1"/>
+    </material>
+    <material name="orange">
+        <color rgba="${255/255} ${108/255} ${10/255} 1.0"/>
+    </material>
+    <material name="brown">
+        <color rgba="${222/255} ${207/255} ${195/255} 1.0"/>
+    </material>
+    <material name="red">
+        <color rgba="0.8 0.0 0.0 1.0"/>
+    </material>
+    <material name="white">
+        <color rgba="1.0 1.0 1.0 1.0"/>
+    </material>
 </robot>

File: mobile_description/urdf/mobile.xacro (robot description, xacro)
@@ -1,59 +1,59 @@
 <?xml version="1.0"?>
 <robot name="mobile" xmlns:xacro="http://www.ros.org/wiki/xacro">
-	<!-- Robot constants and properties -->
-	<xacro:include filename="$(find mobile_description)/urdf/mobile_properties.xacro" />
-	<!-- Import Rviz colors -->
-	<xacro:include filename="$(find mobile_description)/urdf/materials.xacro" />
-	<!-- Gazebo aspects of the robot -->
-	<xacro:include filename="$(find mobile_description)/urdf/mobile.gazebo" />
-	<!-- Inertia matrices -->
-	<xacro:include filename="$(find mobile_description)/urdf/macros.xacro" />
-	<!-- fix the base -->
-	<link name="base_footprint" />
-	<joint name="base_joint" type="fixed">
-		<parent link="base_footprint"/>
-		<child link="chassis"/>
-	</joint>
-	<!-- robot chassis -->
-	<link name="chassis">
-		<inertial>
-			<origin xyz="0 0 ${wheelRadius+0.035}"
-					rpy="0 0 0"/>
-			<mass value="12.0"/>
-			<inertia
-				ixx="0.04680"
-				ixy="0"
-				ixz="-0.00022"
-				iyy="0.07212"
-				iyz="0"
-				izz="0.10440" />
-		</inertial>
-		<visual>
-			<origin xyz="0 0 ${wheelRadius}"
-					rpy="0 0 0"/>
-			<geometry>
-				<mesh filename="package://mobile_description/meshes/chassis.STL" />
-			</geometry>
-			<material name="red"/>
-		</visual>
-		<collision>
-			<origin xyz="0 0 ${wheelRadius}"
-					rpy="0 0 0"/>
-			<geometry>
-				<mesh filename="package://mobile_description/meshes/chassis.STL" />
-			</geometry>
-		</collision>
-	</link>
-	<!-- left-front wheel -->
-	<wheel lr="l" fb="f" Tlr="1" Tfb="1"/>
-	<!-- left-back wheel -->
-	<wheel lr="l" fb="b" Tlr="1" Tfb="-1"/>
-	<!-- right-front wheel -->
-	<wheel lr="r" fb="f" Tlr="-1" Tfb="1"/>
-	<!-- right-back wheel -->
-	<wheel lr="r" fb="b" Tlr="-1" Tfb="-1"/>
-	<!-- Arm models -->
-	<xacro:include filename="$(find mobile_description)/urdf/arm.xacro" />
-	<!-- Sensor models -->
-	<xacro:include filename="$(find mobile_description)/urdf/sensors.xacro" />
+    <!-- Robot constants and properties -->
+    <xacro:include filename="$(find mobile_description)/urdf/mobile_properties.xacro" />
+    <!-- Import Rviz colors -->
+    <xacro:include filename="$(find mobile_description)/urdf/materials.xacro" />
+    <!-- Gazebo aspects of the robot -->
+    <xacro:include filename="$(find mobile_description)/urdf/mobile.gazebo" />
+    <!-- Inertia matrices -->
+    <xacro:include filename="$(find mobile_description)/urdf/macros.xacro" />
+    <!-- fix the base -->
+    <link name="base_footprint" />
+    <joint name="base_joint" type="fixed">
+        <parent link="base_footprint"/>
+        <child link="chassis"/>
+    </joint>
+    <!-- robot chassis -->
+    <link name="chassis">
+        <inertial>
+            <origin xyz="0 0 ${wheelRadius+0.035}"
+                    rpy="0 0 0"/>
+            <mass value="12.0"/>
+            <inertia
+                ixx="0.04680"
+                ixy="0"
+                ixz="-0.00022"
+                iyy="0.07212"
+                iyz="0"
+                izz="0.10440" />
+        </inertial>
+        <visual>
+            <origin xyz="0 0 ${wheelRadius}"
+                    rpy="0 0 0"/>
+            <geometry>
+                <mesh filename="package://mobile_description/meshes/chassis.STL" />
+            </geometry>
+            <material name="red"/>
+        </visual>
+        <collision>
+            <origin xyz="0 0 ${wheelRadius}"
+                    rpy="0 0 0"/>
+            <geometry>
+                <mesh filename="package://mobile_description/meshes/chassis.STL" />
+            </geometry>
+        </collision>
+    </link>
+    <!-- left-front wheel -->
+    <wheel lr="l" fb="f" Tlr="1" Tfb="1"/>
+    <!-- left-back wheel -->
+    <wheel lr="l" fb="b" Tlr="1" Tfb="-1"/>
+    <!-- right-front wheel -->
+    <wheel lr="r" fb="f" Tlr="-1" Tfb="1"/>
+    <!-- right-back wheel -->
+    <wheel lr="r" fb="b" Tlr="-1" Tfb="-1"/>
+    <!-- Arm models -->
+    <xacro:include filename="$(find mobile_description)/urdf/arm.xacro" />
+    <!-- Sensor models -->
+    <xacro:include filename="$(find mobile_description)/urdf/sensors.xacro" />
 </robot>
