Commit message: Added simple gripper, replaced \t's with spaces in all docs.
Signed-off-by: Fatih Kaan AKKUS <fthknakkus@hotmail.com>

File: mobile_description/urdf/mobile_properties.xacro (robot description, xacro)
@@ -1,29 +1,29 @@
 <?xml version="1.0"?>
 <robot xmlns:xacro="http://www.ros.org/wiki/xacro">
-	<!-- Constants -->
-	<xacro:property name="PI" value="3.1415926535897931"/>
-	<!-- Chassis properties -->
-	<xacro:property name="chassisHeight" value="0.10"/>
-	<xacro:property name="chassisLength" value="0.40"/>
-	<xacro:property name="chassisWidth" value="0.27"/>
-	<xacro:property name="chassisMass" value="5.0"/>
-	<!-- Differential-drive wheels properties -->
-	<xacro:property name="wheelWidth" value="0.026"/>
-	<xacro:property name="wheelRadius" value="0.045"/>
-	<xacro:property name="wheelMass" value="0.060"/>
-	<xacro:property name="wheelOffsetY" value="0.037"/>
-	<!-- Hokuyo laser properties -->
-	<xacro:property name="hokuyoMass" value="0.01"/>
-	<xacro:property name="hokuyoLength" value="0.05"/>
-	<xacro:property name="hokuyoWidth" value="0.05"/>
-	<xacro:property name="hokuyoHeight" value="0.07"/>
-	<xacro:property name="hokuyoOffsetX" value="0.17"/>
-	<xacro:property name="hokuyoOffsetZ" value="0.174"/>
-	<!-- Camera properties -->
-	<xacro:property name="cameraLength" value="0.04"/>
-	<xacro:property name="cameraWidth" value="0.08"/>
-	<xacro:property name="cameraHeight" value="0.03"/>
-	<xacro:property name="cameraMass" value="0.01"/>
-	<xacro:property name="cameraOffsetX" value="0.18"/>
-	<xacro:property name="cameraOffsetZ" value="0.1222"/>
+    <!-- Constants -->
+    <xacro:property name="PI" value="3.1415926535897931"/>
+    <!-- Chassis properties -->
+    <xacro:property name="chassisHeight" value="0.10"/>
+    <xacro:property name="chassisLength" value="0.40"/>
+    <xacro:property name="chassisWidth" value="0.27"/>
+    <xacro:property name="chassisMass" value="5.0"/>
+    <!-- Differential-drive wheels properties -->
+    <xacro:property name="wheelWidth" value="0.026"/>
+    <xacro:property name="wheelRadius" value="0.045"/>
+    <xacro:property name="wheelMass" value="0.060"/>
+    <xacro:property name="wheelOffsetY" value="0.037"/>
+    <!-- Hokuyo laser properties -->
+    <xacro:property name="hokuyoMass" value="0.01"/>
+    <xacro:property name="hokuyoLength" value="0.05"/>
+    <xacro:property name="hokuyoWidth" value="0.05"/>
+    <xacro:property name="hokuyoHeight" value="0.07"/>
+    <xacro:property name="hokuyoOffsetX" value="0.17"/>
+    <xacro:property name="hokuyoOffsetZ" value="0.174"/>
+    <!-- Camera properties -->
+    <xacro:property name="cameraLength" value="0.04"/>
+    <xacro:property name="cameraWidth" value="0.08"/>
+    <xacro:property name="cameraHeight" value="0.03"/>
+    <xacro:property name="cameraMass" value="0.01"/>
+    <xacro:property name="cameraOffsetX" value="0.18"/>
+    <xacro:property name="cameraOffsetZ" value="0.1222"/>
 </robot>

File: mobile_description/urdf/sensors.xacro (robot description, xacro)
@@ -51,7 +51,5 @@
               rpy="0 0 0"/>
       <geometry>
-        <box size="${hokuyoLength}
-                   ${hokuyoWidth}
-                   ${hokuyoHeight}"/>
+        <mesh filename="package://mobile_description/meshes/hokuyo.dae"/>
       </geometry>
     </collision>

Commit message: Created go_initial_pose action client.
- Small changes
- Small fixes

Signed-off-by: Fatih Kaan AKKUS <fthknakkus@hotmail.com>

File: mobile_description/urdf/arm.xacro (robot description, xacro)
@@ -362,5 +362,6 @@
                 xyz = "0 0 0"
                 rpy = "0 0 0"/>
-            <mass value="0.05"/>
+            <mass
+                value="0.05"/>
             <inertia
                 ixx="0.000004"
@@ -410,7 +411,8 @@
         <inertial>
             <origin
-                xyz="0 0 0"
-                rpy="0 0 0" />
-            <mass value="0.05"/>
+                xyz="-0.035 0 0.045"
+                rpy="0 0 0" />
+            <mass
+                value="0.05"/>
             <inertia
                 ixx="0.0001"
@@ -458,5 +460,6 @@
                 xyz="0.035 0 0.045"
                 rpy="0 0 0" />
-            <mass value="0.05"/>
+            <mass
+                value="0.05"/>
             <inertia
                 ixx="0.00001"

File: mobile_description/urdf/macros.xacro (robot description, xacro)
@@ -34,5 +34,6 @@
                     xyz="0 0 0.005"
                     rpy="0 0 0" />
-                <mass value="${wheelMass}"/>
+                <mass
+                    value="${wheelMass}"/>
                 <cylinder_inertia
                     m="${wheelMass}"
@@ -73,5 +74,5 @@
             <mu1 value="1.2"/>
             <mu2 value="1.2"/>
-            <kp value="1.0E+6"/>
+            <kp value="1.0E+7"/>
             <kd value="1.0E+0"/>
             <minDepth>0.001</minDepth>

File: mobile_description/urdf/mobile.xacro (robot description, xacro)
@@ -2,5 +2,5 @@
 <robot name="mobile" xmlns:xacro="http://www.ros.org/wiki/xacro">
     <!-- Robot constants and properties -->
-    <xacro:include filename="$(find mobile_description)/urdf/mobile_properties.xacro" />
+    <xacro:include filename="$(find mobile_description)/urdf/properties.xacro" />
     <!-- Import Rviz colors -->
     <xacro:include filename="$(find mobile_description)/urdf/materials.xacro" />
@@ -18,7 +18,9 @@
     <link name="chassis">
         <inertial>
-            <origin xyz="0 0 ${wheelRadius+0.035}"
-                    rpy="0 0 0"/>
-            <mass value="12.0"/>
+            <origin
+                xyz="0 0 ${wheelRadius+0.035}"
+                rpy="0 0 0"/>
+            <mass
+                value="12.0"/>
             <inertia
                 ixx="0.04680"
@@ -30,6 +32,7 @@
         </inertial>
         <visual>
-            <origin xyz="0 0 ${wheelRadius}"
-                    rpy="0 0 0"/>
+            <origin
+                xyz="0 0 ${wheelRadius}"
+                rpy="0 0 0"/>
             <geometry>
                 <mesh filename="package://mobile_description/meshes/chassis.STL" />
@@ -38,6 +41,7 @@
         </visual>
         <collision>
-            <origin xyz="0 0 ${wheelRadius}"
-                    rpy="0 0 0"/>
+            <origin
+                xyz="0 0 ${wheelRadius}"
+                rpy="0 0 0"/>
             <geometry>
                 <mesh filename="package://mobile_description/meshes/chassis.STL" />

File: mobile_description/urdf/properties.xacro (robot description, xacro)
@@ -7,5 +7,5 @@
     <xacro:property name="chassisLength" value="0.40"/>
     <xacro:property name="chassisWidth" value="0.27"/>
-    <xacro:property name="chassisMass" value="5.0"/>
+    <xacro:property name="chassisMass" value="12.0"/>
     <!-- Differential-drive wheels properties -->
     <xacro:property name="wheelWidth" value="0.026"/>

File: mobile_description/urdf/sensors.xacro (robot description, xacro)
@@ -1,74 +1,82 @@
 <?xml version="1.0" ?>
 <robot xmlns:xacro="http://www.ros.org/wiki/xacro">
-  <link name="camera_link">
-    <collision>
-      <origin xyz="0 0 0"
-              rpy="0 0 0"/>
-      <geometry>
-        <box size="${cameraLength}
-                   ${cameraWidth}
-                   ${cameraHeight}"/>
-      </geometry>
-    </collision>
-    <visual>
-      <origin xyz="0 0 0"
-              rpy="0 0 0"/>
-      <geometry>
-        <box size="${cameraLength}
-                   ${cameraWidth}
-                   ${cameraHeight}"/>
-      </geometry>
-      <material name="green"/>
-    </visual>
-    <inertial>
-      <mass value="${cameraMass}" />
-      <origin xyz="0 0 0"
-              rpy="0 0 0"/>
-      <box_inertia m="${cameraMass}"
-                   x="${cameraLength}"
-                   y="${cameraWidth}"
-                   z="${cameraHeight}" />
-    </inertial>
-  </link>
-  <joint name="camera_joint" type="fixed">
-    <axis xyz="0 1 0" />
-    <origin xyz="${cameraOffsetX} 0 ${cameraOffsetZ}"
+    <!-- Camera -->
+    <link name="camera_link">
+        <visual>
+            <origin
+                xyz="0 0 0"
+                rpy="0 0 0"/>
+            <geometry>
+                <box size="${cameraLength} ${cameraWidth} ${cameraHeight}"/>
+            </geometry>
+            <material name="green"/>
+        </visual>
+        <collision>
+            <origin
+                xyz="0 0 0"
+                rpy="0 0 0"/>
+            <geometry>
+                <box size="${cameraLength} ${cameraWidth} ${cameraHeight}"/>
+            </geometry>
+        </collision>
+        <inertial>
+            <origin
+                xyz="0 0 0"
+                rpy="0 0 0"/>
+            <mass
+                value="${cameraMass}" />
+            <box_inertia
+                m="${cameraMass}"
+                x="${cameraLength}"
+                y="${cameraWidth}"
+                z="${cameraHeight}" />
+        </inertial>
+    </link>
+    <joint name="camera_joint" type="fixed">
+        <parent link="chassis"/>
+        <child link="camera_link"/>
+        <origin
+            xyz="${cameraOffsetX} 0 ${cameraOffsetZ}"
             rpy="0 0 0"/>
-    <parent link="chassis"/>
-    <child link="camera_link"/>
-  </joint>
-  <joint name="hokuyo_joint" type="fixed">
-    <axis xyz="0 1 0" />
-    <origin xyz="${hokuyoOffsetX} 0 ${hokuyoOffsetZ}"
+        <axis xyz="0 1 0" />
+    </joint>
+    <!-- Hokuyo Laser -->
+    <link name="hokuyo_link">
+        <collision>
+            <origin
+                xyz="0 0 0"
+                rpy="0 0 0"/>
+            <geometry>
+                <mesh filename="package://mobile_description/meshes/hokuyo.dae"/>
+            </geometry>
+        </collision>
+        <visual>
+            <origin
+                xyz="0 0 0"
+                rpy="0 0 0"/>
+            <geometry>
+                <mesh filename="package://mobile_description/meshes/hokuyo.dae"/>
+            </geometry>
+        </visual>
+        <inertial>
+            <origin
+                xyz="0 0 0"
+                rpy="0 0 0"/>
+            <mass
+                value="${hokuyoMass}" />
+            <box_inertia
+                m="${hokuyoMass}"
+                x="${hokuyoLength}"
+                y="${hokuyoWidth}"
+                z="${hokuyoHeight}"/>
+        </inertial>
+    </link>
+    <joint name="hokuyo_joint" type="fixed">
+        <parent link="chassis"/>
+        <child link="hokuyo_link"/>
+        <origin
+            xyz="${hokuyoOffsetX} 0 ${hokuyoOffsetZ}"
             rpy="0 0 0"/>
-    <parent link="chassis"/>
-    <child link="hokuyo_link"/>
-  </joint>
-  <!-- Hokuyo Laser -->
-  <link name="hokuyo_link">
-    <collision>
-      <origin xyz="0 0 0"
-              rpy="0 0 0"/>
-      <geometry>
-        <mesh filename="package://mobile_description/meshes/hokuyo.dae"/>
-      </geometry>
-    </collision>
-    <visual>
-      <origin xyz="0 0 0"
-              rpy="0 0 0"/>
-      <geometry>
-        <mesh filename="package://mobile_description/meshes/hokuyo.dae"/>
-      </geometry>
-    </visual>
-    <inertial>
-      <mass value="${hokuyoMass}" />
-      <origin xyz="0 0 0"
-              rpy="0 0 0"/>
-      <box_inertia
-        m="${hokuyoMass}"
-        x="${hokuyoLength}"
-        y="${hokuyoWidth}"
-        z="${hokuyoHeight}"/>
-    </inertial>
-  </link>
+        <axis xyz="0 1 0" />
+    </joint>
 </robot>

Commit message: Signed-off-by: Fatih Kaan AKKUS <fthknakkus@hotmail.com>

File: mobile_description/urdf/arm.xacro (robot description, xacro)
@@ -103,8 +103,8 @@
             xyz="0 0 1" />
         <limit
-            effort="6.0"
-            velocity="1.0"
-            lower="${-3.14}"
-            upper="${3.14}" />
+            effort="10.0"
+            velocity="1.0"
+            lower="${-1.60}"
+            upper="${1.60}" />
     </joint>
     <link
@@ -161,5 +161,5 @@
             xyz="0 0 1" />
         <limit
-            effort="6.0"
+            effort="10.0"
             velocity="1.0"
             lower="${-3.14}"
@@ -219,5 +219,5 @@
             xyz="0 0 1" />
         <limit
-            effort="6.0"
+            effort="10.0"
             velocity="1.0"
             lower="${-3.14}"
@@ -277,5 +277,5 @@
             xyz="0 0 1" />
         <limit
-            effort="6.0"
+            effort="10.0"
             velocity="1.0"
             lower="${-3.14}"
@@ -335,5 +335,5 @@
             xyz="0 0 1" />
         <limit
-            effort="6.0"
+            effort="10.0"
             velocity="1.0"
             lower="${-3.14}"
@@ -386,5 +386,5 @@
             xyz="0 0 1" />
         <limit
-            effort="6.0"
+            effort="10.0"
             velocity="1.0"
             lower="${-3.14}"
@@ -435,5 +435,5 @@
             xyz="1 0 0"/>
         <limit
-            effort="6" lower="0" upper="0.03" velocity="1.0"/>
+            effort="10" lower="0" upper="0.03" velocity="1.0"/>
         <dynamics damping="50" friction="1"/>
     </joint>
@@ -481,5 +481,5 @@
             xyz="1 0 0"/>
         <limit
-            effort="6" lower="-0.03" upper="0" velocity="1.0"/>
+            effort="10.0" lower="-0.03" upper="0" velocity="1.0"/>
     </joint>
     <!-- Arm @ Gazebo -->

File: mobile_description/urdf/properties.xacro (robot description, xacro)
@@ -11,5 +11,5 @@
     <xacro:property name="wheelWidth" value="0.026"/>
     <xacro:property name="wheelRadius" value="0.045"/>
-    <xacro:property name="wheelMass" value="0.060"/>
+    <xacro:property name="wheelMass" value="0.12"/>
     <xacro:property name="wheelOffsetY" value="0.037"/>
     <!-- Hokuyo laser properties -->

Commit message: Added damping and friction params to joints.
Signed-off-by: Fatih Kaan AKKUS <fthknakkus@hotmail.com>

File: mobile_description/urdf/arm.xacro (robot description, xacro)
@@ -95,5 +95,5 @@
         <origin
             xyz="0 0 0.018"
-            rpy="9.5272E-17 2.5487E-17 -1.5708" />
+            rpy="9.5272E-17 2.5487E-17 +1.5708" />
         <parent
             link="m_base" />
@@ -104,7 +104,9 @@
         <limit
             effort="10.0"
-            velocity="1.0"
-            lower="${-1.60}"
-            upper="${1.60}" />
+            velocity="2.0"
+            lower="${-3.1416}"
+            upper="${3.1416}" />
+        <dynamics
+            damping="0.1" friction="0.16"/>
     </joint>
     <link
@@ -153,5 +155,5 @@
         <origin
             xyz="0 0 0.055"
-            rpy="1.5708 -1.5708 0" />
+            rpy="1.5708 -1.5708 +0.0001" />
         <parent
             link="m_link_1" />
@@ -159,10 +161,12 @@
             link="m_link_2" />
         <axis
-            xyz="0 0 1" />
+            xyz="0 0 -1" />
         <limit
             effort="10.0"
-            velocity="1.0"
-            lower="${-3.14}"
-            upper="${3.14}"/>
+            velocity="2.0"
+            lower="${0.0}"
+            upper="${1.658}"/>
+        <dynamics
+            damping="0.1" friction="0.16"/>
     </joint>
     <link
@@ -211,5 +215,5 @@
         <origin
             xyz="0.2 0 0"
-            rpy="4.4409E-16 4.5852E-16 -1.7798E-16" />
+            rpy="4.4409E-16 4.5852E-16 +0.0001" />
         <parent
             link="m_link_2" />
@@ -217,10 +221,12 @@
             link="m_link_3" />
         <axis
-            xyz="0 0 1" />
+            xyz="0 0 -1" />
         <limit
             effort="10.0"
-            velocity="1.0"
-            lower="${-3.14}"
-            upper="${3.14}"/>
+            velocity="2.0"
+            lower="${0.0}"
+            upper="${2.2165}"/>
+        <dynamics
+            damping="0.1" friction="0.16"/>
     </joint>
     <link
@@ -269,5 +275,5 @@
         <origin
             xyz="0.2 0 0"
-            rpy="-3.3307E-16 -6.6356E-16 -1.9531E-16" />
+            rpy="-3.3307E-16 -6.6356E-16 +0.0001" />
         <parent
             link="m_link_3" />
@@ -275,10 +281,12 @@
             link="m_link_4" />
         <axis
-            xyz="0 0 1" />
+            xyz="0 0 -1" />
         <limit
             effort="10.0"
-            velocity="1.0"
-            lower="${-3.14}"
-            upper="${3.14}"/>
+            velocity="2.0"
+            lower="${-1.309}"
+            upper="${1.8326}"/>
+        <dynamics
+            damping="0.1" friction="0.16"/>
     </joint>
     <!-- <link
@@ -387,7 +395,9 @@
         <limit
             effort="10.0"
-            velocity="1.0"
+            velocity="2.0"
             lower="${-3.14}"
             upper="${3.14}"/>
+        <dynamics
+            damping="0.1" friction="0.16"/>
     </joint>
     <link name="gripper_finger_left">
@@ -436,5 +446,6 @@
         <limit
             effort="10" lower="0" upper="0.03" velocity="1.0"/>
-        <dynamics damping="50" friction="1"/>
+        <dynamics
+            damping="0.01" friction="0.16"/>
     </joint>
      <link name="gripper_finger_right">
@@ -482,4 +493,6 @@
         <limit
             effort="10.0" lower="-0.03" upper="0" velocity="1.0"/>
+        <dynamics
+            damping="0.01" friction="0.16"/>
     </joint>
     <!-- Arm @ Gazebo -->

Commit message: Update

File: mobile_description/urdf/arm.xacro (robot description, xacro)
@@ -290,62 +290,4 @@
             damping="0.1" friction="0.16"/>
     </joint>
-    <!-- <link
-        name="m_link_gripper">
-        <inertial>
-            <origin
-                xyz="-0.0069546 0.0010309 -0.036727"
-                rpy="0 0 0" />
-            <mass
-                value="0.098787" />
-            <inertia
-                ixx="5.8957E-05"
-                ixy="1.4882E-06"
-                ixz="5.6679E-06"
-                iyy="6.3174E-05"
-                iyz="-4.7843E-07"
-                izz="2.5215E-05" />
-        </inertial>
-        <visual>
-            <origin
-                xyz="0 0 0"
-                rpy="0 0 0" />
-            <geometry>
-                <mesh
-                    filename="package://mobile_description/meshes/m_link_gripper.STL" />
-            </geometry>
-            <material
-                name="">
-                <color
-                    rgba="0.75294 0.75294 0.75294 1" />
-            </material>
-        </visual>
-        <collision>
-            <origin
-                xyz="0 0 0"
-                rpy="0 0 0" />
-            <geometry>
-                <mesh
-                    filename="package://mobile_description/meshes/m_link_gripper.STL" />
-            </geometry>
-        </collision>
-    </link> -->
-    <!-- <joint
-        name="m_joint_5"
-        type="revolute">
-        <origin
-            xyz="0.0895 0 0.0095"
-            rpy="1.5708 3.861E-32 -1.5708" />
-        <parent
-            link="m_link_4" />
-        <child
-            link="m_link_gripper" />
-        <axis
-            xyz="0 0 1" />
-        <limit
-            effort="10.0"
-            velocity="1.0"
-            lower="${-3.14}"
-            upper="${3.14}"/>
-    </joint> -->
     <link name="m_link_gripper">
         <visual>
@@ -445,5 +387,8 @@
             xyz="1 0 0"/>
         <limit
-            effort="10" lower="0" upper="0.03" velocity="1.0"/>
+            effort="10"
+            lower="0"
+            upper="0.03"
+            velocity="1.0"/>
         <dynamics
             damping="0.01" friction="0.16"/>
@@ -492,5 +437,8 @@
             xyz="1 0 0"/>
         <limit
-            effort="10.0" lower="-0.03" upper="0" velocity="1.0"/>
+            effort="10.0"
+            lower="-0.03"
+            upper="0"
+            velocity="1.0"/>
         <dynamics
             damping="0.01" friction="0.16"/>

File: mobile_description/urdf/macros.xacro (robot description, xacro)
@@ -68,6 +68,8 @@
                 xyz="0 0 ${Tlr}"
                 rpy="0 0 0" />
-            <limit effort="100.0" velocity="100.0"/>
-            <joint_properties damping="0.0" friction="0.0"/>
+            <limit
+                effort="100.0"
+                velocity="100.0"/>
+            <dynamics damping="0.0" friction="0.0"/>
         </joint>
         <gazebo reference="w${lr}${fb}">
